File: kicad/carte-prog.kicad_pcb (KiCad board)
At the start: 2 copper layers, 71.1 x 49.8 mm, 14 parts, among them J1 Connecteur côté carte, J2 RJ12 - Côté ordinateur, J3 CHOIX ALIM, J4 DB9_Female, U1 LM1117-3.3, U2 MAX232

Commit message: Correction sens condensateur V-
Parts:
- J2: value RJ12 - Côté ordinateur -> RJ12
- moved C8 2.54 mm to (214.6, 129.5), turned to 90 degrees
Connections:
- C8 pad 1: Net-(C8-Pad1) -> GND
- C8 pad 2: GND -> Net-(C8-Pad2)
- U2 pad 6: Net-(C8-Pad1) -> Net-(C8-Pad2)
Routing:
- net Net-(C8-Pad2): track 0.00 -> 6.77 mm
- net Net-(C8-Pad1): track 6.77 -> 0.00 mm
Other:
- board text added: "v1.1"
- board text removed: "v 1.X"
